Commit message: added gazebo plugins to xacro files

File: src/diff_drive_bot/urdf/robot.urdf.xacro (robot description, xacro)
@@ -1,169 +1,5 @@
-<?xml version="1.0"?>
-<robot xmlns:xacro="http://www.ros.org/wiki/xacro" name="robot">
-<xacro:property name="width" value = "0.4"/>
-<xacro:property name="length" value = "0.6"/>
-<xacro:property name="height" value = "0.2"/>
-<xacro:property name="wheel_radius" value = "0.1"/>
-<xacro:property name="wheel_len" value = "0.05"/>
-<xacro:property name = "caster" value = "0.05"/>
-    <material name="orange">
-        <color rgba="0.6 0.4 0 1"/>
-    </material>
-    <material name = "gray">
-        <color rgba = "0.7 0.7 0.7 1"/>
-    </material>
-    <material name = "white">
-        <color rgba="1 1 1 1"/>
-    </material>
-    <link name = "base_footprint"/>
-    <joint name = "base_joint" type = "fixed">
-        <parent link = "base_footprint"/>
-        <child link = "base_link"/>
-        <origin xyz = "0 0 0.1" rpy = "0 0 0" />
-    </joint>
-    <link name = "base_link">
-        <visual>
-            <geometry>
-                <box size = "${length} ${width} ${height}" />
-            </geometry>
-            <origin xyz = "0 0 0.1" rpy = "0 0 0"/>
-            <material name= "orange"/>
-        </visual>
-        <collision>
-            <geometry>
-                <box size = "${length} ${width} ${height}" />
-            </geometry>
-        </collision>
-        <inertial>
-            <mass value="5"/>
-            <origin xyz="0 0 0" rpy = "0 0 0"/>
-            <inertia ixx="0.083" ixy="0" ixz="0" iyy="0.11" iyz="0" izz="0.13"/>
-        </inertial>
-    </link>
-    <link name = "left_wheel">
-        <visual>
-            <geometry>
-                <cylinder radius = "${wheel_radius}" length = "${wheel_len}"/>
-            </geometry>
-            <origin xyz = "0 0 0" rpy = "1.57 0 0"/>
-            <material name = "gray"/>
-        </visual>
-        <collision>
-            <geometry>
-                <cylinder radius = "${wheel_radius}" length = "${wheel_len}"/>
-            </geometry>
-            <origin xyz = "0 0 0" rpy = "1.57 0 0"/>
-        </collision>
-        <inertial>
-            <mass value="0.5"/>
-            <origin xyz="0 0 0" rpy = "0 0 0"/>
-            <inertia ixx="0.0014" ixy="0" ixz="0" iyy="0.0014" iyz="0" izz="0.0025"/>
-        </inertial>
-    </link>
-    <joint name = "left_wheel_joint" type = "continuous">
-        <parent link = "base_link"/>
-        <child link = "left_wheel"/>
-        <origin xyz = "-${length/4} ${width/2 + wheel_len/2} 0"/>
-        <axis xyz = "0 1 0"/>
-    </joint>
-    <link name = "right_wheel">
-        <visual>
-            <geometry>
-                <cylinder radius = "${wheel_radius}" length = "${wheel_len}"/>
-            </geometry>
-            <origin xyz = "0 0 0" rpy = "1.57 0 0"/>
-            <material name = "gray"/>
-        </visual>
-        <collision>
-            <geometry>
-                <cylinder radius = "${wheel_radius}" length = "${wheel_len}"/>
-            </geometry>
-            <origin xyz = "0 0 0" rpy = "1.57 0 0"/>
-        </collision>
-        <inertial>
-            <mass value="0.5"/>
-            <origin xyz="0 0 0" rpy = "0 0 0"/>
-            <inertia ixx="0.0014" ixy="0" ixz="0" iyy="0.0014" iyz="0" izz="0.0025"/>
-        </inertial>
-    </link>
-    <joint name = "right_wheel_joint" type = "continuous">
-        <parent link = "base_link"/>
-        <child link = "right_wheel"/>
-        <origin xyz = "-${length/4} -${width/2 + wheel_len/2} 0"/>
-        <axis xyz = "0 1 0"/>
-    </joint>
-    <link name = "caster_wheel">
-        <visual>
-            <geometry>
-                <sphere radius = "${caster}"/>
-            </geometry>
-            <origin xyz = "0 0 0" rpy = "0 0 0"/>
-            <material name = "white"/>
-        </visual>
-        <collision>
-            <geometry>
-                <sphere radius = "${caster}"/>
-            </geometry>
-            <origin xyz = "0 0 0" rpy = "0 0 0"/>
-        </collision>
-        <inertial>
-            <mass value="0.2"/>
-            <origin xyz="0 0 0" rpy = "0 0 0"/>
-            <inertia ixx="0.001" ixy="0" ixz="0" iyy="0.001" iyz="0" izz="0.001"/>
-        </inertial>
-    </link>
-    <joint name = "caster_wheel_joint" type = "fixed">
-        <parent link = "base_link"/>
-        <child link = "caster_wheel"/>
-        <origin xyz = "0.2 0 -0.05"/>
-    </joint>
-    <link name = "lidar">
-        <visual>
-            <geometry>
-                <cylinder radius = "0.1" length = "0.05"/>
-            </geometry>
-            <origin xyz = "0 0 0" rpy = "0 0 0"/>
-            <material name = "white"/>
-        </visual>
-        <collision>
-            <geometry>
-                <cylinder radius = "0.1" length = "0.05"/>
-            </geometry>
-            <origin xyz = "0 0 0" rpy = "0 0 0"/>
-        </collision>
-        <inertial>
-            <mass value = "0.1"/>
-            <origin xyz = "0 0 0" rpy = "0 0 0"/>
-            <inertia ixx="0.0005" ixy="0" ixz="0" iyy="0.0005" iyz="0" izz="0.0005"/>
-        </inertial>
-    </link>
-    <joint name = "lidar_joint" type = "fixed">
-        <parent link = "base_link"/>
-        <child link = "lidar"/>
-        <origin xyz = "0 0 0.225" rpy = "0 0 0"/>
-    </joint>
-        <gazebo>
-        <plugin
-            filename="gz-sim-diff-drive-system" name="gz::sim::systems::DiffDrive">
-            <!-- Topic for the command input -->
-            <topic>/cmd_vel</topic>
-            <left_joint>left_wheel_joint</left_joint>
-            <right_joint>right_wheel_joint</right_joint>
-            <wheel_separation>0.45</wheel_separation>
-            <wheel_radius>0.1</wheel_radius>
-            <odom_topic>odom</odom_topic>
-            <frame_id>odom</frame_id>
-            <child_frame_id>base_link</child_frame_id>
-            <odom_publisher_frequency>100</odom_publisher_frequency>
-            <tf_topic>/tf</tf_topic>
-            <max_velocity>3.0</max_velocity>
-            <max_linear_acceleration>10</max_linear_acceleration>
-        </plugin>
-        <plugin
-            filename="gz-sim-joint-state-publisher-system" name="gz::sim::systems::JointStatePublisher">
-            <topic>joint_states</topic>
-            <joint_name>left_wheel_joint</joint_name>
-            <joint_name>right_wheel_joint</joint_name>
-        </plugin>
-    </gazebo>
+<?xml version = "1.0"?>
+<robot xmlsn:xacro="http://www.ros.org/wiki/xacro" name="robot">
+    <xacro:include filename="chassis.xacro" />
+    <xacro:include filename="gazebo.xacro" />
 </robot>
