Commit message: fixed rviz2 launch

File: src/diff_drive_bot/urdf/chassis.xacro (robot description, xacro)
@@ -16,10 +16,13 @@
         <color rgba="1 1 1 1"/>
     </material>
-    <link name = "base_footprint"/>
+    <material name = "black">
+        <color rgba = "0 0 0 1"/>
+    </material>
+    <!-- <link name = "base_footprint"/>
     <joint name = "base_joint" type = "fixed">
         <parent link = "base_footprint"/>
         <child link = "base_link"/>
         <origin xyz = "0 0 0.1" rpy = "0 0 0" />
-    </joint>
+    </joint> -->
     <link name = "base_link">
         <visual>
@@ -143,3 +146,44 @@
         <origin xyz = "0 0 0.225" rpy = "0 0 0"/>
     </joint>
+    <link name = "camera">
+        <visual>
+            <geometry>
+                <box size = "0.01 0.025 0.025"/>
+            </geometry>
+            <origin xyz = "0 0 0" rpy = "0 0 0"/>
+            <material name = "black"/>
+        </visual>
+        <collision>
+            <geometry>
+                <box size = "0.01 0.025 0.025"/>
+            </geometry>
+            <origin xyz = "0 0 0" rpy = "0 0 0"/>
+        </collision>
+        <inertial>
+            <mass value = "0.01"/>
+            <origin xyz = "0 0 0" rpy = "0 0 0"/>
+            <inertia ixx="0.000217" ixy = "0" ixz = "0" iyy = "0.000417" iyz = "0" izz = "0.000217"/>
+        </inertial>
+    </link>
+    <joint name = "camera_joint" type = "fixed">
+        <parent link = "base_link"/>
+        <child link = "camera"/>
+        <origin xyz = "0.305 0 0.2" rpy = "0 0 0"/>
+    </joint>
+    <gazebo reference="base_link">
+        <mu1>1</mu1>
+        <mu2>1</mu2>
+    </gazebo>
+    <gazebo reference="left_wheel">
+        <mu1>1</mu1>
+        <mu2>1</mu2>
+    </gazebo>
+    <gazebo reference="right_wheel">
+        <mu1>1</mu1>
+        <mu2>1</mu2>
+    </gazebo>
+    <gazebo reference="caster_wheel">
+        <mu1>0.000001</mu1>
+        <mu2>0.000001</mu2>
+    </gazebo>
 </robot>

File: src/diff_drive_bot/urdf/gazebo.xacro (robot description, xacro)
@@ -2,12 +2,12 @@
 <robot>
     <gazebo>
-        <!--diff-drive plugin subscribes to /cmd_vel and publishes /odom-->
-        <plugin
-            filename="gz-sim-diff-drive-system" name="gz::sim::systems::DiffDrive">
-            <topic>/cmd_vel</topic>
+        <plugin filename="gz-sim-diff-drive-system" name="gz::sim::systems::DiffDrive">
+            <right_joint>right_wheel_joint</right_joint>
             <left_joint>left_wheel_joint</left_joint>
-            <right_joint>right_wheel_joint</right_joint>
             <wheel_separation>0.45</wheel_separation>
-            <wheel_radius>0.1</wheel_radius>
+            <!-- <wheel_diameter>0.1</wheel_diameter> -->
+            <max_linear_acceleration>10</max_linear_acceleration>
+worlds
+            <topic>cmd_vel</topic>
             <odom_topic>odom</odom_topic>
             <frame_id>odom</frame_id>
@@ -15,12 +15,9 @@
             <odom_publisher_frequency>100</odom_publisher_frequency>
             <tf_topic>/tf</tf_topic>
-            <max_velocity>3.0</max_velocity>
-            <max_linear_acceleration>10</max_linear_acceleration>
         </plugin>
-        <plugin
-            filename="gz-sim-joint-state-publisher-system" name="gz::sim::systems::JointStatePublisher">
+        <plugin filename="gz-sim-joint-state-publisher-system" name="gz::sim::systems::JointStatePublisher">
             <topic>joint_states</topic>
+            <joint_name>right_wheel_joint</joint_name>
             <joint_name>left_wheel_joint</joint_name>
-            <joint_name>right_wheel_joint</joint_name>
         </plugin>
     </gazebo>
@@ -60,3 +57,6 @@
         </sensor>
     </gazebo>
+    <!-- <gazebo reference="camera">
+        <sensor>
+        </sensor> -->
 </robot>

Commit message: added mapping launch file for slam

File: src/diff_drive_bot/urdf/chassis.xacro (robot description, xacro)
@@ -146,4 +146,10 @@
         <origin xyz = "0 0 0.225" rpy = "0 0 0"/>
     </joint>
+    <link name="scan_link" />
+    <joint name="scan_joint" type="fixed">
+        <parent link="base_link"/>
+        <child link="scan_link"/>
+        <origin xyz="0.0 0 0.225" rpy="0 0 0"/>
+    </joint>
     <link name = "camera">
         <visual>

File: src/diff_drive_bot/urdf/gazebo.xacro (robot description, xacro)
@@ -9,21 +9,23 @@
             <max_linear_acceleration>10</max_linear_acceleration>
             <topic>cmd_vel</topic>
+            <update_rate>30</update_rate>
             <odom_topic>odom</odom_topic>
             <frame_id>odom</frame_id>
             <child_frame_id>base_link</child_frame_id>
-            <odom_publisher_frequency>100</odom_publisher_frequency>
+            <odom_publisher_frequency>30</odom_publisher_frequency>
             <tf_topic>/tf</tf_topic>
         </plugin>
-        <plugin filename="gz-sim-joint-state-publisher-system" name="gz::sim::systems::JointStatePublisher">
+        <!-- <plugin filename="gz-sim-joint-state-publisher-system" name="gz::sim::systems::JointStatePublisher">
             <topic>joint_states</topic>
             <joint_name>right_wheel_joint</joint_name>
             <joint_name>left_wheel_joint</joint_name>
-        </plugin>
+        </plugin> -->
     </gazebo>
-    <gazebo reference="lidar">
+    <gazebo reference="scan_link">
         <sensor name = "gpu_lidar" type = "gpu_lidar">
             <pose relative_to="lidar">0 0 0 0 0 0</pose>
             <topic>scan</topic>
             <update_rate>10</update_rate>
+            <gz_frame_id>scan_link</gz_frame_id>
             <lidar>
                 <scan>
@@ -34,10 +36,10 @@
                         <max_angle>3.14156</max_angle>
                     </horizontal>
-                    <vertical>
+                    <!-- <vertical>
                         <samples>1</samples>
                         <resolution>0.01</resolution>
                         <min_angle>0</min_angle>
                         <max_angle>0</max_angle>
-                    </vertical>
+                    </vertical>                        -->
                 </scan>
                 <range>
@@ -51,4 +53,5 @@
                     <stddev>0.01</stddev>
                 </noise>
+                <frame_id>scan_link</frame_id>
             </lidar>
             <always_on>1</always_on>

Commit message: mapped the environment and created localization file

File: src/diff_drive_bot/urdf/chassis.xacro (robot description, xacro)
@@ -30,5 +30,5 @@
                 <box size = "${length} ${width} ${height}" />
             </geometry>
-            <origin xyz = "0 0 0.1" rpy = "0 0 0"/>
+            <origin xyz = "0 0 ${2*wheel_radius}" rpy = "0 0 0"/>
             <material name= "orange"/>
         </visual>
@@ -37,8 +37,9 @@
                 <box size = "${length} ${width} ${height}" />
             </geometry>
+            <origin xyz="0 0 ${2*wheel_radius}"/>
         </collision>
         <inertial>
             <mass value="5"/>
-            <origin xyz="0 0 0" rpy = "0 0 0"/>
+            <origin xyz="0 0 ${wheel_radius + height/2}" rpy = "0 0 0"/>
             <inertia ixx="0.083" ixy="0" ixz="0" iyy="0.11" iyz="0" izz="0.13"/>
         </inertial>
@@ -67,5 +68,5 @@
         <parent link = "base_link"/>
         <child link = "left_wheel"/>
-        <origin xyz = "-${length/4} ${width/2 + wheel_len/2} 0"/>
+        <origin xyz="-${length/4} ${width/2 + wheel_len/2} ${wheel_radius}"/>
         <axis xyz = "0 1 0"/>
     </joint>
@@ -93,5 +94,5 @@
         <parent link = "base_link"/>
         <child link = "right_wheel"/>
-        <origin xyz = "-${length/4} -${width/2 + wheel_len/2} 0"/>
+        <origin xyz = "-${length/4} -${width/2 + wheel_len/2} ${wheel_radius}"/>
         <axis xyz = "0 1 0"/>
     </joint>
@@ -119,5 +120,5 @@
         <parent link = "base_link"/>
         <child link = "caster_wheel"/>
-        <origin xyz = "0.2 0 -0.05"/>
+        <origin xyz = "0.2 0 ${wheel_radius/2}"/>
     </joint>
     <link name = "lidar">
@@ -144,5 +145,5 @@
         <parent link = "base_link"/>
         <child link = "lidar"/>
-        <origin xyz = "0 0 0.225" rpy = "0 0 0"/>
+        <origin xyz = "0 0 ${3*wheel_radius + 0.025}" rpy = "0 0 0"/>
     </joint>
     <link name="scan_link" />
@@ -150,5 +151,5 @@
         <parent link="base_link"/>
         <child link="scan_link"/>
-        <origin xyz="0.0 0 0.225" rpy="0 0 0"/>
+        <origin xyz="0.0 0 ${3*wheel_radius + 0.025}" rpy="0 0 0"/>
     </joint>
     <link name = "camera">

File: src/diff_drive_bot/urdf/gazebo.xacro (robot description, xacro)
@@ -6,5 +6,5 @@
             <left_joint>left_wheel_joint</left_joint>
             <wheel_separation>0.45</wheel_separation>
-            <!-- <wheel_diameter>0.1</wheel_diameter> -->
+            <wheel_radius>0.1</wheel_radius>
             <max_linear_acceleration>10</max_linear_acceleration>
             <topic>cmd_vel</topic>
@@ -15,10 +15,12 @@
             <odom_publisher_frequency>30</odom_publisher_frequency>
             <tf_topic>/tf</tf_topic>
+            <publish_tf>true</publish_tf>
+            <update_rate>50</update_rate>
         </plugin>
-        <!-- <plugin filename="gz-sim-joint-state-publisher-system" name="gz::sim::systems::JointStatePublisher">
+        <plugin filename="gz-sim-joint-state-publisher-system" name="gz::sim::systems::JointStatePublisher">
             <topic>joint_states</topic>
             <joint_name>right_wheel_joint</joint_name>
             <joint_name>left_wheel_joint</joint_name>
-        </plugin> -->
+        </plugin>
     </gazebo>
     <gazebo reference="scan_link">
